File: PDF/Muscolo.sch (KiCad schematic (older format))
At the start: 8 parts

Commit message: Schematic near cmplete
Scheamtic near comlete, deciding whether or not to integrate a STM32
chip onboard ofr integrated PID control on the driver, we'll see.
Parts:
- added C?: VJ0603Y333KXQCW1BC, OnHand-Components:C0603, symbol VJ0603Y333KXQCW1BC
- added C?: C0603C104K5RACTU, OnHand-Components:C0805, symbol C0603C104K5RACTU
- added C? (x4): EEE-1VA101XP, OnHand-Components:EEE-1VA101XP, symbol EEE-1VA101XP
- added Q?: IRFR3707ZPBF, OnHand-Components:IRFR3707ZPBF, symbol IRFR3707ZPBF
- added R? (x2): RC2012F305CS, OnHand-Components:R0603, symbol RC2012F305CS
- added R?: ERJ-3EKF1001V, OnHand-Components:R0603, symbol ERJ-3EKF1001V
Connections:
- net labels added: +12V, CS, OUTA, OUTB
- wire segments 25 -> 38
